Commit message: feat: add reproducible Tancho v2 Isaac Lab training workflow

File: Tancho_v2/Tancho_v2.urdf (robot description, URDF)
Before this commit: robot Tancho_v2, 10 links, 9 joints
Joints:
- joint joint_calf_L: limit lower=-1.57 upper=1.57 effort=10 velocity=5 -> lower=0 upper=3 effort=10 velocity=5
- joint joint_calf_R: limit lower=-1.57 upper=1.57 effort=10 velocity=5 -> lower=0 upper=3 effort=10 velocity=5

File: Tancho_v2_simready/source/stackforce_simready_tancho_v2_lab/stackforce_simready_tancho_v2_lab/assets/robots/Tancho_v2/urdf/Tancho_v2.urdf (robot description, URDF)
Before this commit: robot Tancho_v2, 10 links, 9 joints
Joints:
- joint joint_calf_L: limit lower=-1.57 upper=1.57 effort=10 velocity=5 -> lower=0 upper=3 effort=12.5 velocity=12.5663706
- joint joint_calf_R: limit lower=-1.57 upper=1.57 effort=10 velocity=5 -> lower=0 upper=3 effort=12.5 velocity=12.5663706
- joint joint_thigh_L: limit lower=-1.57 upper=1.57 effort=10 velocity=5 -> lower=-1.57 upper=1.57 effort=12.5 velocity=12.5663706
- joint joint_thigh_R: limit lower=-1.57 upper=1.57 effort=10 velocity=5 -> lower=-1.57 upper=1.57 effort=12.5 velocity=12.5663706
- joint joint_wheel_L: limit lower=-3.14 upper=3.14 effort=10 velocity=5 -> effort=0.45 velocity=52.3598776; type revolute -> continuous
- joint joint_wheel_R: limit lower=-3.14 upper=3.14 effort=10 velocity=5 -> effort=0.45 velocity=52.3598776; type revolute -> continuous
